File: HPE_FlexibleLOM_adapter_x4.kicad_pcb (KiCad board)
At the start: 4 copper layers, 79.2 x 21.7 mm, 5 parts, among them J1 Connector_PCIe_x8, J2 HPE_FlexibleLOM_x8

Commit message: Do layout
Parts:
- added JP3: Jumper_3_Bridged12, Jumper:SolderJumper-3_P1.3mm_Bridged12_Pad1.0x1.5mm, B.Cu at (108.5, 109.8)
- added JP4: Jumper_3_Bridged12, Jumper:SolderJumper-3_P1.3mm_Bridged12_Pad1.0x1.5mm, F.Cu at (104.8, 109.8)
- added R2: 100kR, Resistor_SMD:R_0402_1005Metric, B.Cu at (112.2, 109.2)
- R1: value 10kR -> 100kR; moved to B.Cu
- moved JP1 46.0 mm to (114.5, 109.8), turned to 180 degrees
- moved JP2 43.3 mm to (98.0, 107.0), turned to 180 degrees
- moved R1 19.6 mm to (105.0, 109.2), turned to 90 degrees
Connections:
- J1 pad A1: +12V -> Net-(J1-PadA1)
- J1 pad A10: +3V3 -> Net-(J1-PadA10)
- J1 pad A11: Net-(J1-PadA11) -> /~PERST
- J1 pad A12: Net-(J1-PadA12) -> GND
- J1 pad A13: Net-(J1-PadA13) -> /REFCLK+
- J1 pad A14: /TX0+ -> /REFCLK-
- J1 pad A15: /TX0- -> GND
- J1 pad A16: Net-(J1-PadA16) -> /RX0+
- J1 pad A17: Net-(J1-PadA17) -> /RX0-
- J1 pad A18: Net-(J1-PadA18) -> GND
- J1 pad A19: /TX1+ -> Net-(J1-PadA19)
- J1 pad A20: /TX1- -> GND
- J1 pad A21: Net-(J1-PadA21) -> /RX1+
- J1 pad A22: Net-(J1-PadA22) -> /RX1-
- J1 pad A23: /TX2+ -> GND
- J1 pad A24: /TX2- -> GND
- J1 pad A25: Net-(J1-PadA25) -> /RX2+
- J1 pad A26: Net-(J1-PadA26) -> /RX2-
- J1 pad A27: /TX3+ -> GND
- J1 pad A28: /TX3- -> GND
- J1 pad A29: Net-(J1-PadA29) -> /RX3+
- J1 pad A30: Net-(J1-PadA30) -> /RX3-
- J1 pad A31: Net-(J1-PadA31) -> GND
- J1 pad A33: /TX4+ -> Net-(J1-PadA33)
- J1 pad A34: /TX4- -> GND
- J1 pad A35: Net-(J1-PadA35) -> /RX4+
- J1 pad A36: Net-(J1-PadA36) -> /RX4-
- J1 pad A37: /TX5+ -> GND
- J1 pad A38: /TX5- -> GND
- J1 pad A39: Net-(J1-PadA39) -> /RX5+
- J1 pad A4: Net-(J1-PadA4) -> GND
- J1 pad A40: Net-(J1-PadA40) -> /RX5-
- J1 pad A41: /TX6+ -> GND
- J1 pad A42: /TX6- -> GND
- J1 pad A43: Net-(J1-PadA43) -> /RX6+
- J1 pad A44: Net-(J1-PadA44) -> /RX6-
- J1 pad A45: /TX7+ -> GND
- J1 pad A46: /TX7- -> GND
- J1 pad A47: Net-(J1-PadA47) -> /RX7+
- J1 pad A48: Net-(J1-PadA48) -> /RX7-
- J1 pad A49: Net-(J1-PadA49) -> GND
- J1 pad B1: Net-(J1-PadB1) -> +12V
- J1 pad B10: Net-(J1-PadB10) -> +3V3
- J1 pad B11: /~PERST -> Net-(J1-PadB11)
- J1 pad B13: /REFCLK+ -> GND
- J1 pad B14: /REFCLK- -> /TX0+
- J1 pad B15: Net-(J1-PadB15) -> /TX0-
- J1 pad B16: /RX0+ -> GND
- J1 pad B17: /RX0- -> Net-(J1-PadB17)
- J1 pad B18: Net-(J1-PadB18) -> GND
- J1 pad B19: Net-(J1-PadB19) -> /TX1+
- J1 pad B20: Net-(J1-PadB20) -> /TX1-
- J1 pad B21: /RX1+ -> GND
- J1 pad B22: /RX1- -> GND
- J1 pad B23: Net-(J1-PadB23) -> /TX2+
- J1 pad B24: Net-(J1-PadB24) -> /TX2-
- J1 pad B25: /RX2+ -> GND
- J1 pad B26: /RX2- -> GND
- J1 pad B27: Net-(J1-PadB27) -> /TX3+
- J1 pad B28: Net-(J1-PadB28) -> /TX3-
- J1 pad B29: /RX3+ -> GND
- J1 pad B30: /RX3- -> Net-(J1-PadB30)
- J1 pad B31: Net-(J1-PadB31) -> /PRSNT_x4
- J1 pad B32: Net-(J1-PadB32) -> GND
- J1 pad B33: Net-(J1-PadB33) -> /TX4+
- J1 pad B34: Net-(J1-PadB34) -> /TX4-
- J1 pad B35: /RX4+ -> GND
- J1 pad B36: /RX4- -> GND
- J1 pad B37: Net-(J1-PadB37) -> /TX5+
- J1 pad B38: Net-(J1-PadB38) -> /TX5-
- J1 pad B39: /RX5+ -> GND
- J1 pad B4: Net-(J1-PadB4) -> GND
- J1 pad B40: /RX5- -> GND
- J1 pad B41: Net-(J1-PadB41) -> /TX6+
- J1 pad B42: Net-(J1-PadB42) -> /TX6-
- J1 pad B43: /RX6+ -> GND
- J1 pad B44: /RX6- -> GND
- J1 pad B45: Net-(J1-PadB45) -> /TX7+
- J1 pad B46: Net-(J1-PadB46) -> /TX7-
- J1 pad B47: /RX7+ -> GND
- J1 pad B48: /RX7- -> /PRSNT_x8
- J1 pad B49: Net-(J1-PadB49) -> GND
- J1 pad B7: Net-(J1-PadB7) -> GND
- J2 pad A13: Net-(J2-PadA13) -> GND
- J2 pad A15: Net-(J2-PadA15) -> GND
- J2 pad A16: Net-(J2-PadA16) -> /REFCLK+
- J2 pad A17: /RX0+ -> /REFCLK-
- J2 pad A18: /RX0- -> GND
- J2 pad A19: Net-(J2-PadA19) -> /TX0+
- J2 pad A20: Net-(J2-PadA20) -> /TX0-
- J2 pad A21: /RX1+ -> GND
- J2 pad A22: /RX1- -> GND
- J2 pad A23: Net-(J2-PadA23) -> /TX1+
- J2 pad A24: Net-(J2-PadA24) -> /TX1-
- J2 pad A25: /RX2+ -> GND
- J2 pad A26: /RX2- -> GND
- J2 pad A27: Net-(J2-PadA27) -> /TX2+
- J2 pad A28: Net-(J2-PadA28) -> /TX2-
- J2 pad A29: /RX3+ -> GND
- J2 pad A30: /RX3- -> GND
- J2 pad A31: Net-(J2-PadA31) -> /TX3+
- J2 pad A32: Net-(J2-PadA32) -> /TX3-
- J2 pad A33: /RX4+ -> GND
- J2 pad A34: /RX4- -> GND
- J2 pad A35: Net-(J2-PadA35) -> /TX4+
- J2 pad A36: Net-(J2-PadA36) -> /TX4-
- J2 pad A37: /RX5+ -> GND
- J2 pad A38: /RX5- -> GND
- J2 pad A39: Net-(J2-PadA39) -> /TX5+
- J2 pad A40: Net-(J2-PadA40) -> /TX5-
- J2 pad A41: /RX6+ -> GND
- J2 pad A42: /RX6- -> GND
- J2 pad A43: Net-(J2-PadA43) -> /TX6+
- J2 pad A44: Net-(J2-PadA44) -> /TX6-
- J2 pad A45: /RX7+ -> GND
- J2 pad A46: /RX7- -> GND
- J2 pad A47: Net-(J2-PadA47) -> /TX7+
- J2 pad A48: Net-(J2-PadA48) -> /TX7-
- J2 pad A49: Net-(J2-PadA49) -> GND
- J2 pad A5: Net-(J2-PadA5) -> GND
- J2 pad A8: Net-(J2-PadA8) -> GND
- J2 pad B1: /~PERST -> Net-(J2-PadB1)
- J2 pad B13: Net-(J2-PadB13) -> GND
- J2 pad B16: /REFCLK+ -> GND
- J2 pad B17: /REFCLK- -> /RX0+
- J2 pad B18: Net-(J2-PadB18) -> /RX0-
- J2 pad B19: /TX0+ -> GND
- J2 pad B20: /TX0- -> GND
- J2 pad B21: Net-(J2-PadB21) -> /RX1+
- J2 pad B22: Net-(J2-PadB22) -> /RX1-
- J2 pad B23: /TX1+ -> GND
- J2 pad B24: /TX1- -> GND
- J2 pad B25: Net-(J2-PadB25) -> /RX2+
- J2 pad B26: Net-(J2-PadB26) -> /RX2-
- J2 pad B27: /TX2+ -> GND
- J2 pad B28: /TX2- -> GND
- J2 pad B29: Net-(J2-PadB29) -> /RX3+
- J2 pad B30: Net-(J2-PadB30) -> /RX3-
- J2 pad B31: /TX3+ -> GND
- J2 pad B32: /TX3- -> GND
- J2 pad B33: Net-(J2-PadB33) -> /RX4+
- J2 pad B34: Net-(J2-PadB34) -> /RX4-
- J2 pad B35: /TX4+ -> GND
- J2 pad B36: /TX4- -> GND
- J2 pad B37: Net-(J2-PadB37) -> /RX5+
- J2 pad B38: Net-(J2-PadB38) -> /RX5-
- J2 pad B39: /TX5+ -> GND
- J2 pad B40: /TX5- -> GND
- J2 pad B41: Net-(J2-PadB41) -> /RX6+
- J2 pad B42: Net-(J2-PadB42) -> /RX6-
- J2 pad B43: /TX6+ -> GND
- J2 pad B44: /TX6- -> GND
- J2 pad B45: Net-(J2-PadB45) -> /RX7+
- J2 pad B46: Net-(J2-PadB46) -> /RX7-
- J2 pad B47: /TX7+ -> GND
- J2 pad B48: /TX7- -> GND
- JP1 pad 2: Net-(J2-PadA10) -> Net-(J2-PadB10)
- JP2 pad 2: Net-(J2-PadA1) -> Net-(J2-PadB1)
- R1 pad 1: +3V3 -> Net-(J2-PadA1)
- R1 pad 2: Net-(J2-PadB14) -> +3V3
Routing:
- net /PRSNT_x8: track 0.00 -> 77.2 mm, vias 0 -> 2
- net /PRSNT_x4: track 0.00 -> 54.4 mm, vias 0 -> 2
- net /RX4-: track 0.00 -> 36.3 mm, vias 0 -> 1
- net /RX4+: track 0.00 -> 36.3 mm, vias 0 -> 1
- net /RX3-: track 0.00 -> 35.2 mm, vias 0 -> 1
- net /RX3+: track 0.00 -> 35.2 mm, vias 0 -> 1
- net /RX2-: track 0.00 -> 35.2 mm, vias 0 -> 1
- net /RX2+: track 0.00 -> 35.2 mm, vias 0 -> 1
- net /RX5-: track 0.00 -> 35.1 mm, vias 0 -> 1
- net /RX5+: track 0.00 -> 35.1 mm, vias 0 -> 1
- net /RX6-: track 0.00 -> 34.8 mm, vias 0 -> 1
- net /RX6+: track 0.00 -> 34.8 mm, vias 0 -> 1
- net /RX7-: track 0.00 -> 34.0 mm, vias 0 -> 1
- net /RX7+: track 0.00 -> 34.0 mm, vias 0 -> 1
- net /RX1-: track 0.00 -> 34.0 mm, vias 0 -> 1
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- added copper zone on B.Cu, net +12V
- added copper zone on F.Cu, net +12V
- added copper zone on GND1, net +12V
- added copper zone on B.Cu, net GND
- added copper zone on F.Cu, net GND
- added copper zone on GND1, net GND
- added copper zone on GND2, net GND
Other:
- board text added: "3v3 aux"
- board text added: "Vdet"
- board text added: "lanes"
- board text added: "x4"
- board text added: "x8"
- board text added: "~PERST"
