File: HPE_FlexibleLOM_adapter_x4.sch (KiCad schematic (older format))
At the start: 9 parts, among them J1 Connector_PCIe_x8, J2 HPE_FlexibleLOM_x8

Commit message: RevB
Parts:
- removed JP1, JP2: Jumper_NC_Small, Jumper:SolderJumper-2_P1.3mm_Bridged_Pad1.0x1.5mm, symbol Device:Jumper_NC_Small
- removed JP3: Jumper_3_Bridged12, Jumper:SolderJumper-3_P1.3mm_Bridged12_Pad1.0x1.5mm, symbol Jumper:Jumper_3_Bridged12
- removed R1: 100kR, Resistor_SMD:R_0402_1005Metric, symbol Device:R
Connections:
- net +3V3: now also J2.A1 (PWROK), J2.B10 (+3v3_aux)
- net ~PERST: now also J2.A14 (~PERST), R2.1
- no-connect marks 17 -> 18
Other:
- moved on the sheet: R2
Changed lines of the file:
@@
 Wire Wire Line
 	9400 2400 9400 2500
-Wire Wire Line
-	7600 2200 7600 2300
-$Comp
-L Device:Jumper_NC_Small JP2
-U 1 1 5F5FC3C0
-P 7750 2300
-F 0 "JP2" H 7750 2512 50  0000 C CNN
-F 1 "Jumper_NC_Small" H 7750 2421 50  0000 C CNN
-F 2 "Jumper:SolderJumper-2_P1.3mm_Bridged_Pad1.0x1.5mm" H 7750 2300 50  0001 C CNN
-F 3 "~" H 7750 2300 50  0001 C CNN
-	1    7750 2300
-	1    0    0    -1
-$EndComp
-Wire Wire Line
-	7850 2300 7900 2300
-Wire Wire Line
-	7650 2300 7600 2300
-Connection ~ 7600 2300
-Wire Wire Line
-	7600 2300 7600 2400
 $Comp
 L power:+3V3 #PWR0105
@@
 Wire Wire Line
 	7350 2200 7350 3200
-$Comp
-L Device:Jumper_NC_Small JP1
-U 1 1 5F60319F
-P 7600 3200
-F 0 "JP1" H 7600 3412 50  0000 C CNN
-F 1 "Jumper_NC_Small" H 7600 3321 50  0000 C CNN
-F 2 "Jumper:SolderJumper-2_P1.3mm_Bridged_Pad1.0x1.5mm" H 7600 3200 50  0001 C CNN
-F 3 "~" H 7600 3200 50  0001 C CNN
-	1    7600 3200
-	1    0    0    -1
-$EndComp
-Wire Wire Line
-	7700 3200 7900 3200
 Text Label 7500 3900 0    50   ~ 0
 RX0+
@@
 Wire Wire Line
 	9500 3900 9100 3900
-Wire Wire Line
-	9100 2300 10000 2300
-Text Label 10450 3000 2    50   ~ 0
-~PERST
 Wire Wire Line
 	5100 3300 5500 3300
@@
 NoConn ~ 7900 3700
 $Comp
-L Device:R R1
-U 1 1 5F65E582
-P 10000 2100
-F 0 "R1" V 9793 2100 50  0000 C CNN
-F 1 "100kR" V 9884 2100 50  0000 C CNN
-F 2 "Resistor_SMD:R_0402_1005Metric" V 9930 2100 50  0001 C CNN
-F 3 "~" H 10000 2100 50  0001 C CNN
-	1    10000 2100
-	-1   0    0    1
-$EndComp
-$Comp
-L power:+3V3 #PWR0107
-U 1 1 5F66232B
-P 10000 1900
-F 0 "#PWR0107" H 10000 1750 50  0001 C CNN
-F 1 "+3V3" H 10015 2073 50  0000 C CNN
-F 2 "" H 10000 1900 50  0001 C CNN
-F 3 "" H 10000 1900 50  0001 C CNN
-	1    10000 1900
-	1    0    0    -1
-$EndComp
-$Comp
 L power:GND #PWR0108
 U 1 1 5F6950E5
@@
 	7250 7000 7250 7250
 Wire Wire Line
-	7500 3200 7350 3200
-Wire Wire Line
 	7250 6600 7900 6600
 Wire Wire Line
@@
 	9650 3000 9650 3500
 $Comp
-L Jumper:Jumper_3_Bridged12 JP3
-U 1 1 5F9F18D3
-P 10000 3000
-F 0 "JP3" V 9850 2750 50  0000 L CNN
-F 1 "Jumper_3_Bridged12" V 10100 2100 50  0000 L CNN
-F 2 "Jumper:SolderJumper-3_P1.3mm_Bridged12_Pad1.0x1.5mm" H 10000 3000 50  0001 C CNN
-F 3 "~" H 10000 3000 50  0001 C CNN
-	1    10000 3000
-	0    -1   1    0
-$EndComp
-Wire Wire Line
-	10150 3000 10450 3000
-Wire Wire Line
-	10000 3250 10000 3600
-Wire Wire Line
-	9100 3600 9750 3600
-Wire Wire Line
-	10000 2750 10000 2300
-Wire Wire Line
-	10000 1900 10000 1950
-Wire Wire Line
-	10000 2250 10000 2300
-Connection ~ 10000 2300
-$Comp
 L Device:R R2
 U 1 1 5FAB6150
-P 9750 3350
-F 0 "R2" V 9543 3350 50  0000 C CNN
-F 1 "100kR" V 9634 3350 50  0000 C CNN
-F 2 "Resistor_SMD:R_0402_1005Metric" V 9680 3350 50  0001 C CNN
-F 3 "~" H 9750 3350 50  0001 C CNN
-	1    9750 3350
+P 9850 3350
+F 0 "R2" V 9643 3350 50  0000 C CNN
+F 1 "100kR" V 9734 3350 50  0000 C CNN
+F 2 "Resistor_SMD:R_0402_1005Metric" V 9780 3350 50  0001 C CNN
+F 3 "~" H 9850 3350 50  0001 C CNN
+	1    9850 3350
 	-1   0    0    1
 $EndComp
@@
 L power:+3V3 #PWR0112
 U 1 1 5FAB6156
-P 9750 3150
-F 0 "#PWR0112" H 9750 3000 50  0001 C CNN
-F 1 "+3V3" H 9765 3323 50  0000 C CNN
-F 2 "" H 9750 3150 50  0001 C CNN
-F 3 "" H 9750 3150 50  0001 C CNN
-	1    9750 3150
+P 9850 3150
+F 0 "#PWR0112" H 9850 3000 50  0001 C CNN
+F 1 "+3V3" H 9865 3323 50  0000 C CNN
+F 2 "" H 9850 3150 50  0001 C CNN
+F 3 "" H 9850 3150 50  0001 C CNN
+	1    9850 3150
 	1    0    0    -1
 $EndComp
 Wire Wire Line
-	9750 3150 9750 3200
-Wire Wire Line
-	9750 3500 9750 3600
-Connection ~ 9750 3600
-Wire Wire Line
-	9750 3600 10000 3600
+	9850 3150 9850 3200
+Wire Wire Line
+	9850 3500 9850 3600
 $Comp
 L Jumper:Jumper_3_Bridged12 JP4
@@
 Connection ~ 7250 3500
 NoConn ~ 7900 7100
+$Comp
+L power:+3V3 #PWR0107
+U 1 1 5FF4224D
+P 9150 2200
+F 0 "#PWR0107" H 9150 2050 50  0001 C CNN
+F 1 "+3V3" H 9165 2373 50  0000 C CNN
+F 2 "" H 9150 2200 50  0001 C CNN
+F 3 "" H 9150 2200 50  0001 C CNN
+	1    9150 2200
+	1    0    0    -1
+$EndComp
+Wire Wire Line
+	9150 2200 9150 2300
+Wire Wire Line
+	9150 2300 9100 2300
+Wire Wire Line
+	7600 2200 7600 2400
+Wire Wire Line
+	7350 3200 7900 3200
+Text Label 10300 3600 2    50   ~ 0
+~PERST
+Connection ~ 9850 3600
+Wire Wire Line
+	9850 3600 10300 3600
+Wire Wire Line
+	9100 3600 9850 3600
+NoConn ~ 7900 2300
 $EndSCHEMATC

Commit message: Update to experimental RevC
This recision connects some software defined pins to +3v3, some
more pins of unknown function and parts of the NC-SI interface
to GND. At least the latter should not be required to make any
FlexibleLOM card work. The impact of the former two needs to be
determined empirically.
Connections:
- net +3V3: now also J1.A10 (+3v3), J1.A9 (+3v3), J2.A10 (SDP1), J2.A11 (SDP0); no longer J1.B10 (+3v3_aux), J2.B10 (+3v3_aux)
- net GND: now also J2.A4 (NCSI_CLK), J2.A6 (NCSI_TX0), J2.A7 (NCSI_TX1), J2.B11 (?), J2.B9 (NCSI_TX_EN)
- net ~WAKE: now reaches J1.B11 (~WAKE)
- net ~WAKE: now also J2.A9 (~WAKE)
- new net 3v3_aux: J1.B10 (+3v3_aux), J2.B10 (+3v3_aux)
- no-connect marks 18 -> 10
Other:
- moved on the sheet: R2
Changed lines of the file:
@@
 Wire Wire Line
 	9400 2400 9400 2500
-$Comp
-L power:+3V3 #PWR0105
-U 1 1 5F5FF2E2
-P 3350 2200
-F 0 "#PWR0105" H 3350 2050 50  0001 C CNN
-F 1 "+3V3" H 3365 2373 50  0000 C CNN
-F 2 "" H 3350 2200 50  0001 C CNN
-F 3 "" H 3350 2200 50  0001 C CNN
-	1    3350 2200
-	1    0    0    -1
-$EndComp
-Wire Wire Line
-	3350 2200 3350 3200
-Wire Wire Line
-	3350 3200 3900 3200
-$Comp
-L power:+3V3 #PWR0106
-U 1 1 5F6012FD
-P 7350 2200
-F 0 "#PWR0106" H 7350 2050 50  0001 C CNN
-F 1 "+3V3" H 7365 2373 50  0000 C CNN
-F 2 "" H 7350 2200 50  0001 C CNN
-F 3 "" H 7350 2200 50  0001 C CNN
-	1    7350 2200
-	1    0    0    -1
-$EndComp
-Wire Wire Line
-	7350 2200 7350 3200
 Text Label 7500 3900 0    50   ~ 0
 RX0+
@@
 NoConn ~ 7900 2900
 NoConn ~ 7900 3000
-NoConn ~ 7900 3100
-NoConn ~ 9100 2600
-NoConn ~ 9100 2800
-NoConn ~ 9100 2900
-NoConn ~ 9100 3100
-NoConn ~ 9100 3200
-NoConn ~ 9100 3300
 NoConn ~ 9100 3400
-NoConn ~ 7900 3300
 NoConn ~ 7900 3400
 NoConn ~ 7900 3600
@@
 	9650 2700 9100 2700
 Wire Wire Line
-	9650 2700 9650 3000
+	9650 2700 9650 2800
 Wire Wire Line
 	9100 3500 9650 3500
@@
 L Device:R R2
 U 1 1 5FAB6150
-P 9850 3350
-F 0 "R2" V 9643 3350 50  0000 C CNN
-F 1 "100kR" V 9734 3350 50  0000 C CNN
-F 2 "Resistor_SMD:R_0402_1005Metric" V 9780 3350 50  0001 C CNN
-F 3 "~" H 9850 3350 50  0001 C CNN
-	1    9850 3350
+P 10350 3350
+F 0 "R2" V 10143 3350 50  0000 C CNN
+F 1 "100kR" V 10234 3350 50  0000 C CNN
+F 2 "Resistor_SMD:R_0402_1005Metric" V 10280 3350 50  0001 C CNN
+F 3 "~" H 10350 3350 50  0001 C CNN
+	1    10350 3350
 	-1   0    0    1
 $EndComp
@@
 L power:+3V3 #PWR0112
 U 1 1 5FAB6156
-P 9850 3150
-F 0 "#PWR0112" H 9850 3000 50  0001 C CNN
-F 1 "+3V3" H 9865 3323 50  0000 C CNN
-F 2 "" H 9850 3150 50  0001 C CNN
-F 3 "" H 9850 3150 50  0001 C CNN
-	1    9850 3150
+P 10350 3150
+F 0 "#PWR0112" H 10350 3000 50  0001 C CNN
+F 1 "+3V3" H 10365 3323 50  0000 C CNN
+F 2 "" H 10350 3150 50  0001 C CNN
+F 3 "" H 10350 3150 50  0001 C CNN
+	1    10350 3150
 	1    0    0    -1
 $EndComp
 Wire Wire Line
-	9850 3150 9850 3200
-Wire Wire Line
-	9850 3500 9850 3600
+	10350 3150 10350 3200
+Wire Wire Line
+	10350 3500 10350 3600
 $Comp
 L Jumper:Jumper_3_Bridged12 JP4
@@
 	7900 2800 7250 2800
 Wire Wire Line
-	7250 2800 7250 3500
+	7250 2800 7250 3100
 Connection ~ 7250 3500
 NoConn ~ 7900 7100
-$Comp
-L power:+3V3 #PWR0107
-U 1 1 5FF4224D
-P 9150 2200
-F 0 "#PWR0107" H 9150 2050 50  0001 C CNN
-F 1 "+3V3" H 9165 2373 50  0000 C CNN
-F 2 "" H 9150 2200 50  0001 C CNN
-F 3 "" H 9150 2200 50  0001 C CNN
-	1    9150 2200
+Wire Wire Line
+	7600 2200 7600 2400
+Wire Wire Line
+	7350 3200 7900 3200
+Text Label 10800 3600 2    50   ~ 0
+~PERST
+Connection ~ 10350 3600
+Wire Wire Line
+	10350 3600 10800 3600
+NoConn ~ 7900 2300
+Wire Wire Line
+	5100 3100 5400 3100
+Wire Wire Line
+	5400 3100 5400 2950
+Wire Wire Line
+	5100 3200 5400 3200
+Wire Wire Line
+	5400 3200 5400 3100
+Connection ~ 5400 3100
+Text Label 7350 3200 0    50   ~ 0
+3v3_aux
+Text Label 3500 3200 0    50   ~ 0
+3v3_aux
+$Comp
+L power:+3V3 #PWR0105
+U 1 1 60319A8A
+P 5400 2950
+F 0 "#PWR0105" H 5400 2800 50  0001 C CNN
+F 1 "+3V3" H 5415 3123 50  0000 C CNN
+F 2 "" H 5400 2950 50  0001 C CNN
+F 3 "" H 5400 2950 50  0001 C CNN
+	1    5400 2950
 	1    0    0    -1
 $EndComp
-Wire Wire Line
-	9150 2200 9150 2300
-Wire Wire Line
-	9150 2300 9100 2300
-Wire Wire Line
-	7600 2200 7600 2400
-Wire Wire Line
-	7350 3200 7900 3200
-Text Label 10300 3600 2    50   ~ 0
-~PERST
-Connection ~ 9850 3600
-Wire Wire Line
-	9850 3600 10300 3600
-Wire Wire Line
-	9100 3600 9850 3600
-NoConn ~ 7900 2300
+Text Label 3500 3300 0    50   ~ 0
+~WAKE
+Wire Wire Line
+	9100 3100 9500 3100
+Text Label 9500 3100 2    50   ~ 0
+~WAKE
+Wire Wire Line
+	7900 3100 7250 3100
+Connection ~ 7250 3100
+Wire Wire Line
+	7250 3100 7250 3300
+Wire Wire Line
+	7900 3300 7250 3300
+Connection ~ 7250 3300
+Wire Wire Line
+	7250 3300 7250 3500
+Wire Wire Line
+	9100 2600 9650 2600
+Wire Wire Line
+	9650 2600 9650 2700
+Connection ~ 9650 2700
+Wire Wire Line
+	9100 2800 9650 2800
+Connection ~ 9650 2800
+Wire Wire Line
+	9650 2800 9650 2900
+Wire Wire Line
+	9100 2900 9650 2900
+Connection ~ 9650 2900
+Wire Wire Line
+	9650 2900 9650 3000
+Wire Wire Line
+	9100 3600 10350 3600
+Wire Wire Line
+	9100 3200 9750 3200
+Wire Wire Line
+	9750 3200 9750 2300
+Wire Wire Line
+	9100 2300 9750 2300
+Connection ~ 9750 2300
+Wire Wire Line
+	9750 2300 9750 2200
+$Comp
+L power:+3V3 #PWR?
+U 1 1 60428F63
+P 9750 2200
+F 0 "#PWR?" H 9750 2050 50  0001 C CNN
+F 1 "+3V3" H 9765 2373 50  0000 C CNN
+F 2 "" H 9750 2200 50  0001 C CNN
+F 3 "" H 9750 2200 50  0001 C CNN
+	1    9750 2200
+	1    0    0    -1
+$EndComp
+Wire Wire Line
+	9750 3300 9750 3200
+Wire Wire Line
+	9100 3300 9750 3300
+Connection ~ 9750 3200
+Wire Wire Line
+	3500 3200 3900 3200
+Wire Wire Line
+	3500 3300 3900 3300
 $EndSCHEMATC
